File: circuit/starbie.kicad_pcb (KiCad board)
At the start: 2 copper layers, 112 x 102 mm, 13 parts, among them J1 Conn_01x04_Pin, J2 Conn_01x08_Pin, SW1 SW_Push, SW2 SW_Push, SW3 SW_Push, U1 XIAO-ESP32-S3-Plus-SMD, U2 DHT11

Commit message: Upload new files for Starbiez
Parts:
- removed U2: DHT11, Sensor:Aosong_DHT11_5.5x12.0_P2.54mm
- added DHT1: DHT, Connector_PinSocket_2.54mm:PinSocket_1x04_P2.54mm_Vertical, F.Cu at (222.6, 49.5)
- R3: value 100k -> 10k
Connections:
- net /DHT11 DATA renamed /DHT DATA
Other:
- board text added: "(o. O;)"
- board text added: "----"
- board text added: "-------------------"
- board text added: ":3"
- board text added: "D/O"
- board text added: "NIL"
- board text added: "endless possibilities"
- board text added: "have fun hacking together with friends"
- board text added: "students!"
