File: circuit/starbie.kicad_pcb (KiCad board)
At the start: 2 copper layers, 112 x 102 mm, 13 parts, among them J1 Conn_01x04_Pin, J2 Conn_01x08_Pin, SW1 SW_Push, SW2 SW_Push, SW3 SW_Push, U1 XIAO-ESP32-S3-Plus-SMD

Commit message: Clean up and new changes
Parts:
- added REF**: MountingHole_2mm, MountingHole:MountingHole_2mm, F.Cu at (177.0, 72.5)
- added REF**: MountingHole_2mm, MountingHole:MountingHole_2mm, F.Cu at (236.0, 118.5)
- added REF**: MountingHole_2mm, MountingHole:MountingHole_2mm, F.Cu at (190.0, 107.5)
- added REF**: MountingHole_2mm, MountingHole:MountingHole_2mm, F.Cu at (219.0, 35.5)
