File: circuit/starbie.kicad_sch (KiCad schematic)
At the start: 13 parts, among them J1 Conn_01x04_Pin, J2 Conn_01x08_Pin, SW1 SW_Push, SW2 SW_Push, SW3 SW_Push, U1 XIAO-ESP32-S3-Plus-SMD, U2 DHT11

Commit message: Upload new files for Starbiez
Parts:
- removed U2: DHT11, Sensor:Aosong_DHT11_5.5x12.0_P2.54mm, symbol Sensor:DHT11
- added J3: DHT, Connector_PinSocket_2.54mm:PinSocket_1x04_P2.54mm_Vertical, symbol Connector:Conn_01x04_Pin
- R3: value 100k -> 10k
Connections:
- net +3V3: now also J3.1 (Pin_1)
- net GND: now also J3.4 (Pin_4)
- net DHT11 DATA renamed DHT DATA
- net DHT DATA: now also J3.2 (Pin_2)
- no-connect marks 12 -> 13
Other:
- note added: "- oh my god, the DHT11, DHT21 and DHT22 are interchangeable with pinouts! - expandibility time!"
- moved on the sheet: R1

Commit message: Clean up and new changes
Other:
- note added: "- oh my, the DHT11, DHT21 and DHT22 are interchangeable with pinouts! - expandibility time!"
- note removed: "- oh my god, the DHT11, DHT21 and DHT22 are interchangeable with pinouts! - expandibility time!"
Changed lines of the file:
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@@
 		)
 	)
-	(text "- oh my god, the DHT11, DHT21 and DHT22 are interchangeable with pinouts!\n- expandibility time!"
+	(text "- oh my, the DHT11, DHT21 and DHT22 are interchangeable with pinouts!\n- expandibility time!"
 		(exclude_from_sim no)
 		(at 170.434 76.708 0)
